File: untitled_4.brd (EAGLE design)
At the start: 100 x 93.2 mm, 98 parts, among them IC1 LM1875T, IC2 LM1875T, IC3 LM1875T, IC4 LM1875T, IC5 NE5532N, IC6 NE5532N, J2 power, J3 audio_output, J4 B3P-VH(LF)(SN), J5 +25v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

Commit message: 后级放大:更新
Parts:
- added J7: B3P-VH(LF)(SN), Connectors:HDR-03
- moved C27 12.6 mm to (5.07, 21.3)
- moved C17 9.71 mm to (4.93, 15.0)
- moved C25 6.42 mm to (8.84, 26.7)
- moved C31 6.10 mm to (3.06, 26.4)
- moved C20 3.91 mm to (14.5, 26.8)
- moved C28 1.02 mm to (20.4, 29.3)
- moved R10 0.51 mm to (10.1, 33.6)
- moved R32 0.51 mm to (10.1, 36.1)
- moved R37 0.51 mm to (10.3, 38.6)
- moved R40 0.51 mm to (10.2, 41.1)
- moved R20 0.51 mm to (10.0, 31.1)
- moved C22 0.40 mm to (3.78, 46.9)
Connections:
- new net N$13: C17.P$2, C20.2, J7.3
- new net N$53: C3.P$1, R2.1, W01.1-2
- net GND: now also J7.2
- net N$16: now also J7.1; no longer C3.P$1, R2.1, W01.1-2
- net N$58: no longer C17.P$2, C20.2
Routing:
- net N$16: track 126.2 -> 28.6 mm
- net N$53: track 0.00 -> 83.6 mm
- net GND: track 433.2 -> 473.7 mm
- net N$58: track 120.4 -> 91.7 mm
- net N$13: track 0.00 -> 26.6 mm
- net N$69: track 13.1 -> 23.6 mm
- net N$68: track 20.1 -> 28.8 mm
- net N$62: track 82.0 -> 75.9 mm
- net N$21: track 90.3 -> 87.1 mm
- net N$61: track 43.7 -> 40.7 mm
- net N$27: track 21.9 -> 19.2 mm
- net N$49: track 19.6 -> 18.1 mm
- net N$8: track 112.9 -> 111.5 mm
- net N$39: track 18.3 -> 17.8 mm
- net N$55: track 9.60 -> 9.10 mm
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Other:
- outline, holes or cut-outs redrawn
