File: 3886/3886-main.brd (EAGLE design)
At the start: 117.3 x 93.2 mm, 18 parts, among them J1 audio_output, J6 audio_output

Commit message: add
Parts:
- moved C10 287.4 mm to (106.2, 61.0)
- moved C9 285.7 mm to (101.6, 72.6)
- moved B1 209.4 mm to (17.8, 76.7), turned to 270 degrees
- moved C5 202.7 mm to (93.0, 83.3), turned to 90 degrees
- moved C6 202.7 mm to (72.6, 83.3), turned to 90 degrees
- moved C7 202.7 mm to (52.3, 83.3), turned to 90 degrees
- moved C8 202.7 mm to (32.0, 83.3), turned to 90 degrees
- moved J1 184.3 mm to (6.10, 80.3), turned to 270 degrees
- moved C1 120.9 mm to (93.0, 63.0), turned to 90 degrees
- moved C2 120.9 mm to (72.6, 63.0), turned to 90 degrees
- moved C3 120.9 mm to (52.3, 63.0), turned to 90 degrees
- moved C4 120.9 mm to (32.0, 63.0), turned to 90 degrees
- moved U$2 22.3 mm to (27.4, 18.8)
- moved U$1 22.3 mm to (28.4, 41.1)
- moved J6 15.6 mm to (109.1, 78.4)
